File: od_pedal_pcb/od_pedal_pcb.kicad_sch (KiCad schematic)
At the start: 30 parts, among them J1 JST_VDD, J3 JST_IN, J4 JST_OUT, U1 TL072

Commit message: feat: changes to bypass
Parts:
- removed R3: 180k, Resistor_THT:R_Axial_DIN0207_L6.3mm_D2.5mm_P10.16mm_Horizontal, symbol Device:R
- renumbered 3PDTB to 3PDTC
Connections:
- net at RV2.2, RV3.1: now also 3PDTA.3 (C)
- net at J4.2 (Pin_2): now also 3PDTA.2 (B); no longer RV3.2
- net at C3.2, C5.1, RV1.1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: now also D1.2 (A), D2.1 (K); no longer 3PDTA.3 (C)
- net at 3PDTA.1 (A): now also C4.1, C9.1, U1.6 (-), U1.7
Other:
- note added: "Selector"
- moved on the sheet: 3PDTC, C1, C2, C3, C4, C5, C6, C7, C8, C9, D1, D2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

Commit message: feat: minor adjustments
Connections:
- net at RV2.2, RV3.1: no longer 3PDTA.3 (C)
- net at RV3.2: now also 3PDTA.3 (C)
Changed lines of the file:
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@@
-	)
-	(junction
-		(at 203.2 111.76)
-		(diameter 0)
-		(color 0 0 0 0)
 	)
 	(junction
@@
 	(wire
 		(pts
-			(xy 209.55 111.76) (xy 203.2 111.76)
-		)
-		(stroke
-			(width 0)
-			(type default)
-		)
-	)
-	(wire
-		(pts
 			(xy 97.79 82.55) (xy 95.25 82.55)
 		)
@@
 	(wire
 		(pts
+			(xy 209.55 115.57) (xy 209.55 116.84)
+		)
+		(stroke
+			(width 0)
+			(type default)
+		)
+	)
+	(wire
+		(pts
 			(xy 26.67 114.3) (xy 29.21 114.3)
 		)
@@
 	(wire
 		(pts
-			(xy 209.55 115.57) (xy 209.55 111.76)
-		)
-		(stroke
-			(width 0)
-			(type default)
-		)
-	)
-	(wire
-		(pts
 			(xy 156.21 67.31) (xy 156.21 82.55)
 		)
@@
 	(wire
 		(pts
+			(xy 209.55 116.84) (xy 207.01 116.84)
+		)
+		(stroke
+			(width 0)
+			(type default)
+		)
+	)
+	(wire
+		(pts
 			(xy 128.27 82.55) (xy 135.89 82.55)
 		)
@@
 	(wire
 		(pts
+			(xy 105.41 137.16) (xy 105.41 139.7)
+		)
+		(stroke
+			(width 0)
+			(type default)
+		)
+	)
+	(wire
+		(pts
+			(xy 105.41 114.3) (xy 135.89 114.3)
+		)
+		(stroke
+			(width 0)
+			(type default)
+		)
+	)
+	(wire
+		(pts
+			(xy 110.49 82.55) (xy 110.49 93.98)
+		)
+		(stroke
+			(width 0)
+			(type default)
+		)
+	)
+	(wire
+		(pts
+			(xy 156.21 96.52) (xy 156.21 92.71)
+		)
+		(stroke
+			(width 0)
+			(type default)
+		)
+	)
+	(wire
+		(pts
+			(xy 105.41 129.54) (xy 105.41 137.16)
+		)
+		(stroke
+			(width 0)
+			(type default)
+		)
+	)
+	(wire
+		(pts
+			(xy 156.21 63.5) (xy 156.21 67.31)
+		)
+		(stroke
+			(width 0)
+			(type default)
+		)
+	)
+	(wire
+		(pts
+			(xy 83.82 161.29) (xy 78.74 161.29)
+		)
+		(stroke
+			(width 0)
+			(type default)
+		)
+	)
+	(wire
+		(pts
 			(xy 217.17 115.57) (xy 209.55 115.57)
 		)
 		(stroke
-			(width 0)
-			(type default)
-		)
-	)
-	(wire
-		(pts
-			(xy 105.41 137.16) (xy 105.41 139.7)
-		)
-		(stroke
-			(width 0)
-			(type default)
-		)
-	)
-	(wire
-		(pts
-			(xy 105.41 114.3) (xy 135.89 114.3)
-		)
-		(stroke
-			(width 0)
-			(type default)
-		)
-	)
-	(wire
-		(pts
-			(xy 110.49 82.55) (xy 110.49 93.98)
-		)
-		(stroke
-			(width 0)
-			(type default)
-		)
-	)
-	(wire
-		(pts
-			(xy 156.21 96.52) (xy 156.21 92.71)
-		)
-		(stroke
-			(width 0)
-			(type default)
-		)
-	)
-	(wire
-		(pts
-			(xy 105.41 129.54) (xy 105.41 137.16)
-		)
-		(stroke
-			(width 0)
-			(type default)
-		)
-	)
-	(wire
-		(pts
-			(xy 156.21 63.5) (xy 156.21 67.31)
-		)
-		(stroke
-			(width 0)
-			(type default)
-		)
-	)
-	(wire
-		(pts
-			(xy 83.82 161.29) (xy 78.74 161.29)
-		)
-		(stroke
